Commit message: PR Feedback

File: c3pzero_description/urdf/c3pzero_base.xacro (robot description, xacro)
@@ -218,13 +218,4 @@
     <origin xyz="0 0 0.19" rpy="0 0 0"/>
   </joint>
-  <!-- ros2 control -->
-  <!-- TODO Uncomment when gz_ros2_control is working -->
-  <!-- <xacro:include filename="$(find c3pzero_description)/urdf/c3pzero_base.ros2_control.xacro" />
-  <xacro:if value="${simulation}">
-    <xacro:property name="ros2_control_name" value="IgnitionSystem"/>
-    <xacro:c3pzero_ros2_control
-      name="${ros2_control_name}"
-      simulation="${simulation}"/>
-  </xacro:if> -->
   <xacro:if value="$(arg simulation)">
     <gazebo reference="lidar_link">
@@ -334,10 +325,4 @@
           <odom_topic>/wheel/odom</odom_topic>
         </plugin>
-        <!-- TODO Uncomment when gz_ros2_control is working -->
-        <!-- <plugin filename="libign_ros2_control-system.so" name="ign_ros2_control">
-          <robot_param>robot_description</robot_param>
-          <robot_param_node>robot_state_publisher</robot_param_node>
-          <parameters>$(find c3pzero_description)/config/c3pzero_controllers.yaml</parameters>
-        </plugin> -->
     </gazebo>
   </xacro:if>

Commit message: add config settings required by Studio to base config package

File: c3pzero_description/urdf/c3pzero_base.xacro (robot description, xacro)
@@ -1,5 +1,5 @@
 <?xml version="1.0"?>
 <robot name="c3pzero" xmlns:xacro="http://ros.org/wiki/xacro">
-  <xacro:property name="simulation" default="true" />
+  <xacro:arg name="simulation" default="true" />
   <!-- Define robot constants -->
   <xacro:property name="base_width" value="0.46"/>

Commit message: Testing changes

File: c3pzero_description/urdf/c3pzero_base.xacro (robot description, xacro)
@@ -216,5 +216,5 @@
     <parent link="base_link"/>
     <child link="lidar_link"/>
-    <origin xyz="0 0 0.19" rpy="0 0 0"/>
+    <origin xyz="0 0 0.19" rpy="0 0 3.14156"/>
   </joint>
   <xacro:if value="$(arg simulation)">
